Commit message: finish section 7

File: ros2_ws/src/my_robot_description/urdf/mobile_base.xacro (robot description, xacro)
@@ -66,5 +66,5 @@
             <origin xyz="0.0 0.0 0.0" rpy="0.0 0.0 0.0"/>
             <geometry>
-                <sphere radius="${2*wheel_radius/2.0}"/>
+                <sphere radius="${wheel_radius/2.0}"/>
             </geometry>
             <material name="grey"/>
@@ -76,5 +76,5 @@
             </geometry>
         </collision>
-        <xacro:sphere_inertia m="0.5" r="${wheel_radius/2.0}"
+        <xacro:sphere_inertia m="0.5" r="${2*wheel_radius/2.0}"
             xyz="0.0 0.0 0.0" rpy="0.0 0.0 0.0"/>
     </link>

File: ros2_ws/src/my_robot_description/urdf/mobile_gazebo_base.xacro (robot description, xacro)
@@ -4,3 +4,33 @@
         <material>Gazebo/Blue</material>
     </gazebo>
+    <gazebo reference="right_wheel_link">
+        <material>Gazebo/Grey</material>
+    </gazebo>
+    <gazebo reference="left_wheel_link">
+        <material>Gazebo/Grey</material>
+    </gazebo>
+    <gazebo reference="caster_wheel_link">
+        <material>Gazebo/Grey</material>
+        <mu1 value="0.1" />
+        <mu2 value="0.2" />
+    </gazebo>
+    <gazebo>
+        <plugin name="diff_drive_control" filename="libgazebo_ros_diff_drive.so">
+            <!-- Update rate in Hz -->
+            <update_rate>50</update_rate>
+            <!-- wheels -->
+            <left_joint>base_left_wheel_joint</left_joint>
+            <right_joint>base_right_wheel_joint</right_joint>
+            <!-- kinematics -->
+            <wheel_separation>0.45</wheel_separation>
+            <wheel_diameter>0.2</wheel_diameter>
+            <!-- output -->
+            <publish_odom>true</publish_odom>
+            <publish_odom_tf>true</publish_odom_tf>
+            <publish_wheel_tf>true</publish_wheel_tf>
+            <odometry_topic>odom</odometry_topic>
+            <odometry_frame>odom</odometry_frame>
+            <robot_base_frame>base_footprint</robot_base_frame>
+        </plugin>
+    </gazebo>
 </robot>
