Commit message: finish project

File: ros2_ws/src/my_robot_description/urdf/common_properties.xacro (robot description, xacro)
@@ -1,39 +1,45 @@
 <?xml version="1.0"?>
-<robot xmlns:xacro="http://www.ros.org/wiki/xacro" >
+<robot xmlns:xacro="http://www.ros.org/wiki/xacro">
     <material name="green">
-        <color rgba="0.0 0.5 0.0 1.0"/>
+        <color rgba="0.0 0.5 0.0 1.0" />
     </material>
     <material name="grey">
-        <color rgba="0.5 0.5 0.5 1.0"/>
+        <color rgba="0.5 0.5 0.5 1.0" />
     </material>
     <material name="blue">
-        <color rgba="0.0 0.0 1.0 1.0"/>
+        <color rgba="0.0 0.0 1.0 1.0" />
     </material>
-<xacro:macro name="box_inertia" params="m l w h xyz rpy">
-    <inertial>
-        <origin xyz="${xyz}" rpy="${rpy}"/>
-        <mass value="${m}"/>
-        <inertia ixx="${(m/12)*(h*h + l*l)}" ixy="0.0" ixz="0.0"
-            iyy="${(m/12) * (w*w + l*l)}" iyz="0.0"
-            izz="${(m/12)*(w*w + h*h)}"/>
-    </inertial>
-</xacro:macro>
-<xacro:macro name="cylinder_inertia" params="m r h xyz rpy">
-    <inertial>
-        <origin xyz="${xyz}" rpy="${rpy}"/>
-        <mass value="${m}"/>
-        <inertia ixx="${(m/12)*(3*r*r + h*h)}" ixy="0.0" ixz="0.0"
-            iyy="${(m/12) * (3*r*r + h*h)}" iyz="0.0"
-            izz="${(m/2)*(r*r)}"/>
-    </inertial>
-</xacro:macro>
-<xacro:macro name="sphere_inertia" params="m r xyz rpy">
-    <inertial>
-        <origin xyz="${xyz}" rpy="${rpy}"/>
-        <mass value="${m}"/>
-        <inertia ixx="${(2/5)* m * r * r}" ixy="0.0" ixz="0.0"
-            iyy="${(2/5)* m * r * r}" iyz="0.0"
-            izz="${(2/5)* m * r * r}"/>
-    </inertial>
-</xacro:macro>
+    <material name="orange">
+        <color rgba="1.0 0.64 0.0 1.0" />
+    </material>
+    <material name="yellow">
+        <color rgba="1.0 1.0 0.0 1.0" />
+    </material>
+    <xacro:macro name="box_inertia" params="m l w h xyz rpy">
+        <inertial>
+            <origin xyz="${xyz}" rpy="${rpy}" />
+            <mass value="${m}" />
+            <inertia ixx="${(m/12)*(h*h + l*l)}" ixy="0.0" ixz="0.0"
+                iyy="${(m/12) * (w*w + l*l)}" iyz="0.0"
+                izz="${(m/12)*(w*w + h*h)}" />
+        </inertial>
+    </xacro:macro>
+    <xacro:macro name="cylinder_inertia" params="m r h xyz rpy">
+        <inertial>
+            <origin xyz="${xyz}" rpy="${rpy}" />
+            <mass value="${m}" />
+            <inertia ixx="${(m/12)*(3*r*r + h*h)}" ixy="0.0" ixz="0.0"
+                iyy="${(m/12) * (3*r*r + h*h)}" iyz="0.0"
+                izz="${(m/2)*(r*r)}" />
+        </inertial>
+    </xacro:macro>
+    <xacro:macro name="sphere_inertia" params="m r xyz rpy">
+        <inertial>
+            <origin xyz="${xyz}" rpy="${rpy}" />
+            <mass value="${m}" />
+            <inertia ixx="${(2/5)* m * r * r}" ixy="0.0" ixz="0.0"
+                iyy="${(2/5)* m * r * r}" iyz="0.0"
+                izz="${(2/5)* m * r * r}" />
+        </inertial>
+    </xacro:macro>
 </robot>

File: ros2_ws/src/my_robot_description/urdf/mobile_base.xacro (robot description, xacro)
@@ -2,85 +2,91 @@
 <robot xmlns:xacro="http://www.ros.org/wiki/xacro">
     <xacro:property name="base_length" value="0.6" />
-    <xacro:property name="base_width" value="0.4"/>
-    <xacro:property name="base_height" value="0.2"/>
-    <xacro:property name="wheel_radius" value="0.1"/>
-    <xacro:property name="wheel_length" value="0.05"/>
-    <link name="base_footprint"/>
+    <xacro:property name="base_width" value="0.4" />
+    <xacro:property name="base_height" value="0.2" />
+    <xacro:property name="wheel_radius" value="0.1" />
+    <xacro:property name="wheel_length" value="0.05" />
+    <link name="base_footprint" />
     <link name="base_link">
         <visual name="">
             <geometry>
-                <box size="${base_length} ${base_width} ${base_height}"/>
+                <box size="${base_length} ${base_width} ${base_height}" />
             </geometry>
-            <origin xyz="0.0 0.0 ${base_height/2.0}" rpy="0.0 0.0 0.0"/>
-            <material name="green"/>
+            <origin xyz="0.0 0.0 ${base_height/2.0}" rpy="0.0 0.0 0.0" />
+            <material name="green" />
         </visual>
         <collision>
             <geometry>
-                <box size="${base_length} ${base_width} ${base_height}"/>
+                <box size="${base_length} ${base_width} ${base_height}" />
             </geometry>
-            <origin xyz="0.0 0.0 ${base_height/2.0}" rpy="0.0 0.0 0.0"/>
+            <origin xyz="0.0 0.0 ${base_height/2.0}" rpy="0.0 0.0 0.0" />
         </collision>
         <xacro:box_inertia m="5.0" l="${2*base_length}" w="${2*base_width}" h="${2*base_height}"
-            xyz="0.0 0.0 ${base_height/2.0}" rpy="0.0 0.0 0.0"/>
+            xyz="0.0 0.0 ${base_height/2.0}" rpy="0.0 0.0 0.0" />
     </link>
     <joint name="base_joint" type="fixed">
-        <parent link="base_footprint"/>
-        <child link="base_link"/>
-        <origin xyz="0.0 0.0 ${wheel_radius}" rpy="0.0 0.0 0.0"/>
+        <parent link="base_footprint" />
+        <child link="base_link" />
+        <origin xyz="0.0 0.0 ${wheel_radius}" rpy="0.0 0.0 0.0" />
     </joint>
     <xacro:macro name="wheel_link" params="prefix">
         <link name="${prefix}_wheel_link">
             <visual name="">
-                <origin xyz="0.0 0.0 0.0" rpy="${pi / 2.0} 0.0 0.0"/>
+                <origin xyz="0.0 0.0 0.0" rpy="${pi / 2.0} 0.0 0.0" />
                 <geometry>
-                    <cylinder radius="${wheel_radius}" length="${wheel_length}"/>
+                    <cylinder radius="${wheel_radius}" length="${wheel_length}" />
                 </geometry>
                 <material name="blue" />
             </visual>
             <collision>
-                <origin xyz="0.0 0.0 0.0" rpy="${pi / 2.0} 0.0 0.0"/>
+                <origin xyz="0.0 0.0 0.0" rpy="${pi / 2.0} 0.0 0.0" />
                 <geometry>
-                    <cylinder radius="${wheel_radius}" length="${wheel_length}"/>
+                    <cylinder radius="${wheel_radius}" length="${wheel_length}" />
                 </geometry>
             </collision>
             <xacro:cylinder_inertia m="1.0" r="${2*wheel_radius}" h="${2*wheel_length}"
-                xyz="0.0 0.0 0.0" rpy="${pi / 2.0} 0.0 0.0"/>
+                xyz="0.0 0.0 0.0" rpy="${pi / 2.0} 0.0 0.0" />
         </link>
     </xacro:macro>
     <xacro:wheel_link prefix="right" />
     <joint name="base_right_wheel_joint" type="continuous">
-        <origin xyz="${-base_length/4.0} ${-(base_width + wheel_length) / 2.0} 0.0" rpy="${pi} 0.0 0.0"/>
-        <parent link="base_link"/>
-        <child link="right_wheel_link"/>
-        <axis xyz="0.0 1.0 0.0"/>
+        <origin xyz="${-base_length/4.0} ${-(base_width + wheel_length) / 2.0} 0.0"
+            rpy="${pi} 0.0 0.0" />
+        <parent link="base_link" />
+        <child link="right_wheel_link" />
+        <axis xyz="0.0 1.0 0.0" />
     </joint>
     <xacro:wheel_link prefix="left" />
     <joint name="base_left_wheel_joint" type="continuous">
-        <origin xyz="${-base_length/4.0} ${(base_width + wheel_length) / 2.0} 0.0" rpy="0.0 0.0 0.0"/>
-        <parent link="base_link"/>
-        <child link="left_wheel_link"/>
-        <axis xyz="0.0 1.0 0.0"/>
+        <origin xyz="${-base_length/4.0} ${(base_width + wheel_length) / 2.0} 0.0" rpy="0.0 0.0 0.0" />
+        <parent link="base_link" />
+        <child link="left_wheel_link" />
+        <axis xyz="0.0 1.0 0.0" />
     </joint>
     <link name="caster_wheel_link">
         <visual>
-            <origin xyz="0.0 0.0 0.0" rpy="0.0 0.0 0.0"/>
+            <origin xyz="0.0 0.0 0.0" rpy="0.0 0.0 0.0" />
             <geometry>
-                <sphere radius="${wheel_radius/2.0}"/>
+                <sphere radius="${wheel_radius/2.0}" />
             </geometry>
-            <material name="grey"/>
+            <material name="grey" />
         </visual>
         <collision>
-            <origin xyz="0.0 0.0 0.0" rpy="0.0 0.0 0.0"/>
+            <origin xyz="0.0 0.0 0.0" rpy="0.0 0.0 0.0" />
             <geometry>
-                <sphere radius="${wheel_radius/2.0}"/>
+                <sphere radius="${wheel_radius/2.0}" />
             </geometry>
         </collision>
         <xacro:sphere_inertia m="0.5" r="${2*wheel_radius/2.0}"
-            xyz="0.0 0.0 0.0" rpy="0.0 0.0 0.0"/>
+            xyz="0.0 0.0 0.0" rpy="0.0 0.0 0.0" />
     </link>
     <joint name="base_caster_joint" type="fixed">
-        <origin xyz="${base_length/3.0} 0.0 ${-wheel_radius/2.0}" rpy="0.0 0.0 0.0"/>
-        <parent link="base_link"/>
-        <child link="caster_wheel_link"/>
+        <origin xyz="${base_length/3.0} 0.0 ${-wheel_radius/2.0}" rpy="0.0 0.0 0.0" />
+        <parent link="base_link" />
+        <child link="caster_wheel_link" />
+    </joint>
+    <joint name="joint_base_arm" type="fixed">
+        <parent link="base_link" />
+        <child link="arm_base_link" />
+        <origin xyz="${base_length/4.0} 0.0 ${base_height}" rpy="0.0 0.0 0.0" />
     </joint>
 </robot>

File: ros2_ws/src/my_robot_description/urdf/my_robot.urdf.xacro (robot description, xacro)
@@ -1,6 +1,8 @@
 <?xml version="1.0"?>
 <robot xmlns:xacro="http://www.ros.org/wiki/xacro" name="my_robot">
-    <xacro:include filename="common_properties.xacro"/>
-    <xacro:include filename="mobile_base.xacro"/>
-    <xacro:include filename="mobile_gazebo_base.xacro"/>
+    <xacro:include filename="common_properties.xacro" />
+    <xacro:include filename="mobile_base.xacro" />
+    <xacro:include filename="mobile_gazebo_base.xacro" />
+    <xacro:include filename="camera.xacro" />
+    <xacro:include filename="arm.xacro" />
 </robot>
